Commit message: 整理 webgui 目录、统一资源路径与中文注释

File: webgui/robot_description/dummy_real_v3/urdf/dummy_real_v3.urdf (robot description, URDF)
Before this commit: robot dummy_real_v3, 11 links, 10 joints
Links:
- link base_link: geometry collision mesh filename=package://dummy_real_v3/meshes/base_link.STL; visual mesh filename=package://dummy_real_v3/meshes/base_link.STL
- link camera_link: geometry collision mesh filename=package://dummy_real_v3/meshes/camera_link.STL; visual mesh filename=package://dummy_real_v3/meshes/camera_link.STL
- link link1: geometry collision mesh filename=package://dummy_real_v3/meshes/link1.STL; visual mesh filename=package://dummy_real_v3/meshes/link1.STL
- link link2: geometry collision mesh filename=package://dummy_real_v3/meshes/link2.STL; visual mesh filename=package://dummy_real_v3/meshes/link2.STL
- link link3: geometry collision mesh filename=package://dummy_real_v3/meshes/link3.STL; visual mesh filename=package://dummy_real_v3/meshes/link3.STL
- link link4: geometry collision mesh filename=package://dummy_real_v3/meshes/link4.STL; visual mesh filename=package://dummy_real_v3/meshes/link4.STL
- link link5: geometry collision mesh filename=package://dummy_real_v3/meshes/link5.STL; visual mesh filename=package://dummy_real_v3/meshes/link5.STL
- link link6: geometry collision mesh filename=package://dummy_real_v3/meshes/link6.STL; visual mesh filename=package://dummy_real_v3/meshes/link6.STL
- link link7: geometry collision mesh filename=package://dummy_real_v3/meshes/link7.STL; visual mesh filename=package://dummy_real_v3/meshes/link7.STL
- link link8: geometry collision mesh filename=package://dummy_real_v3/meshes/link8.STL; visual mesh filename=package://dummy_real_v3/meshes/link8.STL
- link link9: geometry collision mesh filename=package://dummy_real_v3/meshes/link9.STL; visual mesh filename=package://dummy_real_v3/meshes/link9.STL
